File: hardware/verbot.kicad_sch (KiCad schematic)
At the start: 20 parts, among them J1 Raspberry Pi Zero 2 W, J2 5V USB power bank, M1 Pimoroni OnOff SHIM, M2 DRV8833 carrier, M3 Verbot 3V motor, M4 Verbot gearbox harness, M5 MAX98357A I2S DAC, M6 MCP23017 @ 0x20, SW1 stop, SW2 forwards, SW3 reverse, SW4 rotate_left, SW5 rotate_right, SW6 pick_up, SW7 put_down, SW8 talk

Commit message: fix: schematic notes underspecify power pins and keypad polling
POWER note didn't say which of the twelve stacked +5V/+3V3/GND stubs map
to which physical header pins - the stock Raspberry_Pi_2_3 symbol prints
its duplicate power pins on top of each other, so the drawing needs to
spell out the list the netlist already encodes. FRONT PANEL note left
the INTA/INTB no-connects unexplained; add the 50 Hz polling rationale
that previously existed only as a Python comment, matching the design
spec's requirement.

Regenerated verbot.kicad_sch and re-exported the PDF/SVG. ERC still 0
errors, 0 warnings.

Co-Authored-By: Claude Opus 5 <noreply@anthropic.com>
Other:
- note added: "POWER: 5V USB bank -> OnOff SHIM -> Pi 5V rail and DRV8833 VCC. Motor current therefore passes through the SHIM load switch (~2A). Cap VERBOT_ACTION_SPEED near +/-60 and rely on C1 for transients. +5V: pins 2,4 | +3V3: 1,17 | GND: 6,9,14,20,25,30,34,39"
- note removed: "POWER: 5V USB bank -> OnOff SHIM -> Pi 5V rail and DRV8833 VCC. Motor current therefore passes through the SHIM load switch (~2A). Cap VERBOT_ACTION_SPEED near +/-60 and rely on C1 for transients."
Changed lines of the file:
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@@
 		(instances
 			(project "verbot"
-				(path "/7a414ca5-97a5-46b4-9969-fc1e113f1c98" (reference "J1") (unit 1))))
+				(path "/d49374cf-9cc8-4aa0-b7fc-5d8adb057fd4" (reference "J1") (unit 1))))
 	)
 	(symbol
@@
 		(instances
 			(project "verbot"
-				(path "/7a414ca5-97a5-46b4-9969-fc1e113f1c98" (reference "M1") (unit 1))))
+				(path "/d49374cf-9cc8-4aa0-b7fc-5d8adb057fd4" (reference "M1") (unit 1))))
 	)
 	(symbol
@@
 		(instances
 			(project "verbot"
-				(path "/7a414ca5-97a5-46b4-9969-fc1e113f1c98" (reference "J2") (unit 1))))
+				(path "/d49374cf-9cc8-4aa0-b7fc-5d8adb057fd4" (reference "J2") (unit 1))))
 	)
 	(wire (pts (xy 26.67 58.42) (xy 30.48 58.42))
@@
 		(instances
 			(project "verbot"
-				(path "/7a414ca5-97a5-46b4-9969-fc1e113f1c98" (reference "#FLG01") (unit 1))))
+				(path "/d49374cf-9cc8-4aa0-b7fc-5d8adb057fd4" (reference "#FLG01") (unit 1))))
 	)
 	(label "+5V" (at 44.45 105.41 0)
@@
 		(instances
 			(project "verbot"
-				(path "/7a414ca5-97a5-46b4-9969-fc1e113f1c98" (reference "#FLG02") (unit 1))))
+				(path "/d49374cf-9cc8-4aa0-b7fc-5d8adb057fd4" (reference "#FLG02") (unit 1))))
 	)
 	(label "+3V3" (at 82.55 105.41 0)
 		(effects (font (size 1.27 1.27)) (justify left)))
-	(text "POWER: 5V USB bank -> OnOff SHIM -> Pi 5V rail and DRV8833 VCC.\nMotor current therefore passes through the SHIM load switch (~2A).\nCap VERBOT_ACTION_SPEED near +/-60 and rely on C1 for transients." (at 25.4 120.65 0)
+	(text "POWER: 5V USB bank -> OnOff SHIM -> Pi 5V rail and DRV8833 VCC.\nMotor current therefore passes through the SHIM load switch (~2A).\nCap VERBOT_ACTION_SPEED near +/-60 and rely on C1 for transients.\n+5V: pins 2,4 | +3V3: 1,17 | GND: 6,9,14,20,25,30,34,39" (at 25.4 120.65 0)
 		(effects (font (size 1.27 1.27)) (justify left top)))
 	(symbol
@@
 		(instances
 			(project "verbot"
-				(path "/7a414ca5-97a5-46b4-9969-fc1e113f1c98" (reference "M2") (unit 1))))
+				(path "/d49374cf-9cc8-4aa0-b7fc-5d8adb057fd4" (reference "M2") (unit 1))))
 	)
 	(symbol
@@
 		(instances
 			(project "verbot"
-				(path "/7a414ca5-97a5-46b4-9969-fc1e113f1c98" (reference "M3") (unit 1))))
+				(path "/d49374cf-9cc8-4aa0-b7fc-5d8adb057fd4" (reference "M3") (unit 1))))
 	)
 	(symbol
@@
 		(instances
 			(project "verbot"
-				(path "/7a414ca5-97a5-46b4-9969-fc1e113f1c98" (reference "C1") (unit 1))))
+				(path "/d49374cf-9cc8-4aa0-b7fc-5d8adb057fd4" (reference "C1") (unit 1))))
 	)
 	(wire (pts (xy 236.22 166.37) (xy 240.03 166.37))
@@
 		(instances
 			(project "verbot"
-				(path "/7a414ca5-97a5-46b4-9969-fc1e113f1c98" (reference "M4") (unit 1))))
+				(path "/d49374cf-9cc8-4aa0-b7fc-5d8adb057fd4" (reference "M4") (unit 1))))
 	)
 	(wire (pts (xy 295.91 182.88) (xy 292.1 182.88))
@@
 		(instances
 			(project "verbot"
-				(path "/7a414ca5-97a5-46b4-9969-fc1e113f1c98" (reference "M5") (unit 1))))
+				(path "/d49374cf-9cc8-4aa0-b7fc-5d8adb057fd4" (reference "M5") (unit 1))))
 	)
 	(symbol
@@
 		(instances
 			(project "verbot"
-				(path "/7a414ca5-97a5-46b4-9969-fc1e113f1c98" (reference "LS1") (unit 1))))
+				(path "/d49374cf-9cc8-4aa0-b7fc-5d8adb057fd4" (reference "LS1") (unit 1))))
 	)
 	(wire (pts (xy 116.84 210.82) (xy 113.03 210.82))
@@
 		(instances
 			(project "verbot"
-				(path "/7a414ca5-97a5-46b4-9969-fc1e113f1c98" (reference "M6") (unit 1))))
+				(path "/d49374cf-9cc8-4aa0-b7fc-5d8adb057fd4" (reference "M6") (unit 1))))
 	)
 	(wire (pts (xy 69.85 146.05) (xy 66.04 146.05))
@@
 		(instances
 			(project "verbot"
-				(path "/7a414ca5-97a5-46b4-9969-fc1e113f1c98" (reference "SW1") (unit 1))))
+				(path "/d49374cf-9cc8-4aa0-b7fc-5d8adb057fd4" (reference "SW1") (unit 1))))
 	)
 	(wire (pts (xy 35.56 139.7) (xy 31.75 139.7))
@@
 		(instances
 			(project "verbot"
-				(path "/7a414ca5-97a5-46b4-9969-fc1e113f1c98" (reference "SW2") (unit 1))))
+				(path "/d49374cf-9cc8-4aa0-b7fc-5d8adb057fd4" (reference "SW2") (unit 1))))
 	)
 	(wire (pts (xy 35.56 149.86) (xy 31.75 149.86))
@@
 		(instances
 			(project "verbot"
-				(path "/7a414ca5-97a5-46b4-9969-fc1e113f1c98" (reference "SW3") (unit 1))))
+				(path "/d49374cf-9cc8-4aa0-b7fc-5d8adb057fd4" (reference "SW3") (unit 1))))
 	)
 	(wire (pts (xy 35.56 160.02) (xy 31.75 160.02))
@@
 		(instances
 			(project "verbot"
-				(path "/7a414ca5-97a5-46b4-9969-fc1e113f1c98" (reference "SW4") (unit 1))))
+				(path "/d49374cf-9cc8-4aa0-b7fc-5d8adb057fd4" (reference "SW4") (unit 1))))
 	)
 	(wire (pts (xy 35.56 170.18) (xy 31.75 170.18))
@@
 		(instances
 			(project "verbot"
-				(path "/7a414ca5-97a5-46b4-9969-fc1e113f1c98" (reference "SW5") (unit 1))))
+				(path "/d49374cf-9cc8-4aa0-b7fc-5d8adb057fd4" (reference "SW5") (unit 1))))
 	)
 	(wire (pts (xy 35.56 180.34) (xy 31.75 180.34))
@@
 		(instances
 			(project "verbot"
-				(path "/7a414ca5-97a5-46b4-9969-fc1e113f1c98" (reference "SW6") (unit 1))))
+				(path "/d49374cf-9cc8-4aa0-b7fc-5d8adb057fd4" (reference "SW6") (unit 1))))
 	)
 	(wire (pts (xy 35.56 190.5) (xy 31.75 190.5))
@@
 		(instances
 			(project "verbot"
-				(path "/7a414ca5-97a5-46b4-9969-fc1e113f1c98" (reference "SW7") (unit 1))))
+				(path "/d49374cf-9cc8-4aa0-b7fc-5d8adb057fd4" (reference "SW7") (unit 1))))
 	)
 	(wire (pts (xy 35.56 200.66) (xy 31.75 200.66))
@@
 		(instances
 			(project "verbot"
-				(path "/7a414ca5-97a5-46b4-9969-fc1e113f1c98" (reference "SW8") (unit 1))))
+				(path "/d49374cf-9cc8-4aa0-b7fc-5d8adb057fd4" (reference "SW8") (unit 1))))
 	)
 	(wire (pts (xy 35.56 210.82) (xy 31.75 210.82))
@@
 		(instances
 			(project "verbot"
-				(path "/7a414ca5-97a5-46b4-9969-fc1e113f1c98" (reference "R1") (unit 1))))
+				(path "/d49374cf-9cc8-4aa0-b7fc-5d8adb057fd4" (reference "R1") (unit 1))))
 	)
 	(symbol
@@
 		(instances
 			(project "verbot"
-				(path "/7a414ca5-97a5-46b4-9969-fc1e113f1c98" (reference "D1") (unit 1))))
+				(path "/d49374cf-9cc8-4aa0-b7fc-5d8adb057fd4" (reference "D1") (unit 1))))
 	)
 	(wire (pts (xy 138.43 166.37) (xy 142.24 166.37))
@@
 	(no_connect (at 138.43 181.61))
 	(no_connect (at 138.43 184.15))
-	(text "FRONT PANEL - VERIFY BEFORE WIRING.\nThis assumes the eight buttons are INDEPENDENT switches to a common rail.\nThat has NOT been confirmed on the real panel. The original PCB also\ncarried the power switching, so bypass it and solder to the switch\ncontacts directly. Check with a meter first.\n\nGPA0-7 are inputs with MCP23017 pull-ups enabled: ACTIVE LOW.\nButton order above is BUTTON_ORDER in hardware/mcp23017.py and is a\nGUESS - reorder it at bring-up if a button triggers the wrong action.\nR1 330R gives ~5mA from 3V3 through a red LED; MCP23017 sources 25mA.\nGPB1-7 float (driver sets them as inputs) - harmless." (at 12.7 254.0 0)
+	(text "FRONT PANEL - VERIFY BEFORE WIRING.\nThis assumes the eight buttons are INDEPENDENT switches to a common rail.\nThat has NOT been confirmed on the real panel. The original PCB also\ncarried the power switching, so bypass it and solder to the switch\ncontacts directly. Check with a meter first.\n\nGPA0-7 are inputs with MCP23017 pull-ups enabled: ACTIVE LOW.\nButton order above is BUTTON_ORDER in hardware/mcp23017.py and is a\nGUESS - reorder it at bring-up if a button triggers the wrong action.\nR1 330R gives ~5mA from 3V3 through a red LED; MCP23017 sources 25mA.\nGPB1-7 float (driver sets them as inputs) - harmless.\nINTA/INTB are no-connect: Mcp23017Keypad polls GPIOA at 50 Hz instead\nof using the interrupt line." (at 12.7 254.0 0)
 		(effects (font (size 1.27 1.27)) (justify left top)))
 	(no_connect (at 195.58 125.73))
